Commit message: refactor(arm7): rescale service, tests, URDF and demo to Design B (0.675 m chain)
Companion to libpick-ik-core 44e3533: the same four Design B linear constants (base->J2 0.180 m, J2->J4/J4->J6 0.215 m each, tool 0.065 m) land in service/arm7.py (JOINTS + TOOL_OFFSET; limits/velocities/axes unchanged) and in robot_description/arm7.urdf, where the visuals are rebuilt at the new dimensions - 50-60 mm structural links, motor-sized pivot spheres (AK10-9 D110 / AK70-10 D95 / J6 placeholder D76), tool D44 shaft, and effort attributes carrying the J2/J4 rated torques (18 / 8.3 Nm).

Tests: anchor expectations regenerated (zero pose 675 mm; pivot heights 0.180/0.395/0.610 m) and the cross-check targets replaced by the Design B set, 200/100/300 mm (deep fold) and 300/150/300 mm (moderate), in test_api/test_binding plus the service-exact look-at/seed targets. The full-pose orientation-metric test now runs on the deterministic gradient solver against an FK-derived goal - the memetics random population seeding measurably stalls at the seed on large-orientation goals (upstream behavior; noted in HANDOVER section 5). 44/44 green.

Web demo: target sliders x/y -550..550 mm, z 0..650 mm, defaults 300/150/300; camera dist 3.3 -> 1.8 m (presets 1.6-1.8 m, wheel clamp 0.3-3.0 m), look-at height 0.5 -> 0.3 m, ground grid 0.15 m / +/-0.6 m; cross-check hint text and the /health arm label updated. Smoke: /fk zero pose 675 mm, /solve succeeds on both targets (CCD 0.00 mm, gradient 0.8 mm, memetic 0.3 mm), clean no-solve at the ~0.151 m inner boundary.

File: robot_description/arm7.urdf (robot description, URDF)
Before this commit: robot arm7, 9 links, 8 joints
Links:
- link base_link: geometry visual cylinder length=0.18 radius=0.10
- link link1: geometry visual box size=0.08 0.08 0.18
- link link2: geometry visual box size=0.06 0.215 0.06; visual sphere radius=0.055
- link link4: geometry visual box size=0.06 0.215 0.06; visual sphere radius=0.048
- link link6: geometry visual box size=0.06 0.065 0.06; visual sphere radius=0.038
- link tool_link: geometry visual box size=0.005 0.005 0.037; visual box size=0.005 0.037 0.005
Joints:
- joint joint1: limit lower=-3.14159 upper=3.14159 effort=100 velocity=2.17 -> lower=-3.14159 upper=3.14159 effort=87 velocity=2.17
- joint joint2: limit lower=-2.09 upper=2.09 effort=100 velocity=2.17 -> lower=-2.09 upper=2.09 effort=18 velocity=2.17; origin xyz=0 0 0.34 rpy=-1.5707963 0 0 -> xyz=0 0 0.18 rpy=-1.5707963 0 0
- joint joint3: limit lower=-3.14159 upper=3.14159 effort=100 velocity=2.17 -> lower=-3.14159 upper=3.14159 effort=87 velocity=2.17
- joint joint4: limit lower=-2.09 upper=2.09 effort=100 velocity=2.17 -> lower=-2.09 upper=2.09 effort=8.3 velocity=2.17; origin xyz=0 0 0.40 rpy=-1.5707963 0 0 -> xyz=0 0 0.215 rpy=-1.5707963 0 0
- joint joint5: limit lower=-3.14159 upper=3.14159 effort=100 velocity=2.61 -> lower=-3.14159 upper=3.14159 effort=12 velocity=2.61
- joint joint6: limit lower=-2.09 upper=2.09 effort=100 velocity=2.61 -> lower=-2.09 upper=2.09 effort=12 velocity=2.61; origin xyz=0 0 0.40 rpy=-1.5707963 0 0 -> xyz=0 0 0.215 rpy=-1.5707963 0 0
- joint joint7: limit lower=-3.14159 upper=3.14159 effort=100 velocity=2.61 -> lower=-3.14159 upper=3.14159 effort=12 velocity=2.61
- joint tool_offset: origin xyz=0 0 0.126 rpy=0 0 0 -> xyz=0 0 0.065 rpy=0 0 0
